File: Optical_filter_electronics_schematic/Controller_Unit.kicad_sch (KiCad schematic)
At the start: 1 part, among them U3 Nucleo-64_F103RB

Commit message: Update PCB schematic
Connections:
- no-connect marks 0 -> 48
Changed lines of the file:
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@@
 	(generator_version "10.0")
 	(paper "A4")
+	(no_connect
+		(at 152.4 66.04)
+	)
+	(no_connect
+		(at 109.22 53.34)
+	)
+	(no_connect
+		(at 109.22 68.58)
+	)
+	(no_connect
+		(at 109.22 101.6)
+	)
+	(no_connect
+		(at 109.22 109.22)
+	)
+	(no_connect
+		(at 152.4 63.5)
+	)
+	(no_connect
+		(at 109.22 63.5)
+	)
+	(no_connect
+		(at 109.22 88.9)
+	)
+	(no_connect
+		(at 152.4 109.22)
+	)
+	(no_connect
+		(at 109.22 40.64)
+	)
+	(no_connect
+		(at 152.4 38.1)
+	)
+	(no_connect
+		(at 152.4 93.98)
+	)
+	(no_connect
+		(at 109.22 66.04)
+	)
+	(no_connect
+		(at 109.22 99.06)
+	)
+	(no_connect
+		(at 152.4 55.88)
+	)
+	(no_connect
+		(at 152.4 111.76)
+	)
+	(no_connect
+		(at 109.22 38.1)
+	)
+	(no_connect
+		(at 109.22 45.72)
+	)
+	(no_connect
+		(at 152.4 101.6)
+	)
+	(no_connect
+		(at 109.22 106.68)
+	)
+	(no_connect
+		(at 109.22 78.74)
+	)
+	(no_connect
+		(at 109.22 104.14)
+	)
+	(no_connect
+		(at 152.4 124.46)
+	)
+	(no_connect
+		(at 109.22 76.2)
+	)
+	(no_connect
+		(at 152.4 71.12)
+	)
+	(no_connect
+		(at 109.22 71.12)
+	)
+	(no_connect
+		(at 152.4 78.74)
+	)
+	(no_connect
+		(at 152.4 53.34)
+	)
+	(no_connect
+		(at 109.22 55.88)
+	)
+	(no_connect
+		(at 109.22 114.3)
+	)
+	(no_connect
+		(at 109.22 73.66)
+	)
+	(no_connect
+		(at 152.4 73.66)
+	)
+	(no_connect
+		(at 152.4 48.26)
+	)
+	(no_connect
+		(at 152.4 60.96)
+	)
+	(no_connect
+		(at 109.22 43.18)
+	)
+	(no_connect
+		(at 152.4 127)
+	)
+	(no_connect
+		(at 109.22 58.42)
+	)
+	(no_connect
+		(at 109.22 86.36)
+	)
+	(no_connect
+		(at 152.4 88.9)
+	)
+	(no_connect
+		(at 152.4 50.8)
+	)
+	(no_connect
+		(at 109.22 60.96)
+	)
+	(no_connect
+		(at 152.4 45.72)
+	)
+	(no_connect
+		(at 152.4 76.2)
+	)
+	(no_connect
+		(at 152.4 91.44)
+	)
+	(no_connect
+		(at 109.22 111.76)
+	)
+	(no_connect
+		(at 152.4 86.36)
+	)
+	(no_connect
+		(at 152.4 99.06)
+	)
+	(no_connect
+		(at 152.4 58.42)
+	)
 	(wire
 		(pts
