File: Optical_filter_electronics_schematic/Motor_Control_and_ADC.kicad_sch (KiCad schematic)
At the start: 7 parts, among them J7 FILTER MOTOR PINS, U2 ADS1115IDGS, U5 DRV8834

Commit message: Update PCB schematic
Connections:
- no-connect marks 3 -> 5
Changed lines of the file:
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@@
+	)
+	(no_connect
+		(at 118.11 67.31)
 	)
 	(no_connect
@@
 		(at 143.51 101.6)
 	)
+	(no_connect
+		(at 118.11 69.85)
+	)
 	(wire
 		(pts
@@
 	(wire
 		(pts
-			(xy 214.63 77.47) (xy 218.44 77.47)
-		)
-		(stroke
-			(width 0)
-			(type default)
-		)
-	)
-	(wire
-		(pts
 			(xy 138.43 77.47) (xy 158.75 77.47)
 		)
@@
 	(wire
 		(pts
+			(xy 210.82 77.47) (xy 218.44 77.47)
+		)
+		(stroke
+			(width 0)
+			(type default)
+		)
+	)
+	(wire
+		(pts
 			(xy 186.69 39.37) (xy 186.69 45.72)
 		)
@@
 	(wire
 		(pts
+			(xy 210.82 74.93) (xy 218.44 74.93)
+		)
+		(stroke
+			(width 0)
+			(type default)
+		)
+	)
+	(wire
+		(pts
 			(xy 138.43 64.77) (xy 143.51 64.77)
 		)
@@
 		(pts
 			(xy 140.97 59.69) (xy 138.43 59.69)
-		)
-		(stroke
-			(width 0)
-			(type default)
-		)
-	)
-	(wire
-		(pts
-			(xy 214.63 74.93) (xy 218.44 74.93)
 		)
 		(stroke
@@
 		)
 	)
-	(label "POT-"
-		(at 214.63 77.47 180)
-		(effects
-			(font
-				(size 1.27 1.27)
-			)
-			(justify right bottom)
-		)
-	)
-	(label "POT+"
-		(at 214.63 74.93 180)
-		(effects
-			(font
-				(size 1.27 1.27)
-			)
-			(justify right bottom)
-		)
-	)
 	(label "GND"
 		(at 213.36 80.01 180)
@@
 			)
 			(justify left bottom)
+		)
+	)
+	(hierarchical_label "POT+"
+		(shape bidirectional)
+		(at 210.82 74.93 180)
+		(effects
+			(font
+				(size 1.27 1.27)
+			)
+			(justify right)
 		)
 	)
@@
 		(effects
 			(font
+				(size 1.27 1.27)
+			)
+			(justify right)
+		)
+	)
+	(hierarchical_label "POT-"
+		(shape bidirectional)
+		(at 210.82 77.47 180)
+		(effects
+			(font

Commit message: changed layout components
Parts:
- C8, C9: footprint Capacitor_THT:C_Disc_D5.0mm_W2.5mm_P2.50mm -> Capacitor_SMD:C_0805_2012Metric_Pad1.18x1.45mm_HandSolder
- R1: footprint Resistor_THT:R_Axial_DIN0207_L6.3mm_D2.5mm_P10.16mm_Horizontal -> Resistor_SMD:R_0805_2012Metric_Pad1.20x1.40mm_HandSolder
Changed lines of the file:
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@@
 			)
 		)
-		(property "Footprint" "Capacitor_THT:C_Disc_D5.0mm_W2.5mm_P2.50mm"
+		(property "Footprint" "Capacitor_SMD:C_0805_2012Metric_Pad1.18x1.45mm_HandSolder"
 			(at 187.6552 53.34 0)
 			(hide yes)
@@
 			)
 		)
-		(property "Footprint" "Resistor_THT:R_Axial_DIN0207_L6.3mm_D2.5mm_P10.16mm_Horizontal"
+		(property "Footprint" "Resistor_SMD:R_0805_2012Metric_Pad1.20x1.40mm_HandSolder"
 			(at 189.992 92.71 90)
 			(hide yes)
@@
 			)
 		)
-		(property "Footprint" "Capacitor_THT:C_Disc_D5.0mm_W2.5mm_P2.50mm"
+		(property "Footprint" "Capacitor_SMD:C_0805_2012Metric_Pad1.18x1.45mm_HandSolder"
 			(at 192.7352 124.46 0)
 			(hide yes)
