File: Optical_filter_electronics_schematic/Optical_filter_electronics_schematic.kicad_pcb (KiCad board)
At the start: 2 copper layers, 242.2 x 90 mm, 24 parts, among them J1 Conn_01x08_Socket, J2 Adafruit_USB_C_Breakout_4090, J7 FILTER MOTOR PINS, U1 ER_OLEDM0.91_1x-I2C, U2 ADS1115IDGS, U3 Nucleo-64_F103RB, U4 AMS1117-3.3, U5 DRV8834

Commit message: Update PCB schematic
Connections:
- J7 pad 6: /Motor_Control_modules/POT+ -> /3.3V
- J7 pad 7: /Motor_Control_modules/POT- -> GND
Routing:
- net /3.3V: track 235.8 -> 266.2 mm
- net Net-(D1-A1): track 21.1 -> 31.7 mm
- net GND: track 0.00 -> 2.00 mm

Commit message: changed layout components
Parts:
- C3, C5: footprint Capacitor_THT:C_Disc_D5.0mm_W2.5mm_P2.50mm -> Capacitor_SMD:C_0805_2012Metric_Pad1.18x1.45mm_HandSolder; moved to B.Cu
- C4, C6: footprint Capacitor_THT:CP_Radial_D5.0mm_P2.00mm -> Capacitor_SMD:C_1206_3216Metric_Pad1.33x1.80mm_HandSolder; moved to B.Cu
- C8, C9: footprint Capacitor_THT:C_Disc_D5.0mm_W2.5mm_P2.50mm -> Capacitor_SMD:C_0805_2012Metric_Pad1.18x1.45mm_HandSolder
- D1, J7: moved to B.Cu
- F1: footprint Fuse:Fuse_Bourns_MF-RG1000 -> Fuse:Fuse_1812_4532Metric_Pad1.30x3.40mm_HandSolder; moved to B.Cu
- R1, R2, R3, R4, R5: footprint Resistor_THT:R_Axial_DIN0207_L6.3mm_D2.5mm_P10.16mm_Horizontal -> Resistor_SMD:R_0805_2012Metric_Pad1.20x1.40mm_HandSolder
- moved D2 181.5 mm to (72.0, 112.2), turned to -90 degrees
- moved D3 176.1 mm to (70.8, 78.0), turned to 90 degrees
- moved R4 152.2 mm to (70.2, 120.2)
- moved J1 147.1 mm to (97.6, 158.0)
- moved R5 137.7 mm to (71.5, 70.2), turned to 180 degrees
- moved C8 96.1 mm to (70.8, 31.8)
- moved C7 95.7 mm to (69.8, 25.4)
- moved J7 91.1 mm to (145.2, 53.8), turned to 180 degrees
- moved R3 81.4 mm to (106.0, 118.5), turned to 90 degrees
- moved U3 81.0 mm to (69.4, 63.5), turned to -90 degrees
- moved U5 72.6 mm to (70.2, 49.5), turned to 90 degrees
- moved R2 71.5 mm to (109.2, 118.5), turned to -90 degrees
- moved J2 56.1 mm to (72.0, 96.0)
- moved U4 50.4 mm to (87.8, 97.4)
- moved C3 49.6 mm to (88.5, 113.5)
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Routing:
- net /3.3V: track 266.2 -> 0.00 mm, vias 2 -> 0
- net /Controller_Unit/PC1: track 141.8 -> 0.00 mm, vias 1 -> 0
- net /PB9: track 124.4 -> 0.00 mm, vias 1 -> 0
- net /Controller_Unit/PB8: track 116.0 -> 0.00 mm, vias 1 -> 0
- net /5V: track 111.4 -> 0.00 mm
- net /Controller_Unit/PB0: track 111.0 -> 0.00 mm, vias 1 -> 0
- net /Controller_Unit/PA3: track 102.8 -> 0.00 mm, vias 1 -> 0
- net /Controller_Unit/PA2: track 89.0 -> 0.00 mm
- net Net-(J7-Pin_5): track 84.7 -> 0.00 mm, vias 1 -> 0
- net /Controller_Unit/PB11: track 66.2 -> 0.00 mm
- net /Controller_Unit/PA4: track 64.1 -> 0.00 mm, vias 1 -> 0
- net /Controller_Unit/PB10: track 60.0 -> 0.00 mm, vias 1 -> 0
- net /Controller_Unit/PB12: track 57.9 -> 0.00 mm, vias 1 -> 0
- net /Controller_Unit/PB1: track 55.9 -> 0.00 mm
- net /Controller_Unit/PB15: track 49.8 -> 0.00 mm
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- removed copper zone on B.Cu, net GND
- removed copper zone on F.Cu, net GND
Other:
- board size 242.2 x 90 mm -> 92 x 179.2 mm
